File: hardware/BME280.sch (KiCad schematic (older format))
At the start: 1 part

Commit message: add MPNs and datasheet links to components
Parts:
- U?: MPN (none) -> BME280
Changed lines of the file:
@@
 F 1 "BME280" H 6100 4225 60  0000 C CNN
 F 2 "" H 6100 4225 60  0001 C CNN
-F 3 "" H 6100 4225 60  0001 C CNN
+F 3 "https://ae-bst.resource.bosch.com/media/_tech/media/datasheets/BST-BME280-DS002.pdf" H 6100 4225 60  0001 C CNN
+F 4 "BME280" H 6100 4225 60  0001 C CNN "MPN"
 	1    6100 4225
 	1    0    0    -1
