File: hardware/DA14682.sch (KiCad schematic (older format))
At the start: 0 parts

Commit message: add MPNs and datasheet links to components
Other:
- note added: "datasheet for DA14682\n\nTODO: create sch symbol and footprint for DA14682\n\nhttps://www.dialog-semiconductor.com/sites/default/files/da14682_ds_3v1.pdf"
Changed lines of the file:
@@
 $Descr A4 11693 8268
 encoding utf-8
-Sheet 1 6
+Sheet 4 6
 Title ""
 Date ""
@@
 Comment4 ""
 $EndDescr
+Text Notes 4125 3775 0    60   ~ 0
+datasheet for DA14682\n\nTODO: create sch symbol and footprint for DA14682\n\nhttps://www.dialog-semiconductor.com/sites/default/files/da14682_ds_3v1.pdf
 $EndSCHEMATC
