File: hardware/display.sch (KiCad schematic (older format))
At the start: 1 part

Commit message: add MPNs and datasheet links to components
Parts:
- U?: MPN (none) -> AML130A2402A
Changed lines of the file:
@@
 F 1 "AML130A2402A" H 6100 4550 60  0000 C CNN
 F 2 "" H 6075 4625 60  0001 C CNN
-F 3 "" H 6075 4625 60  0001 C CNN
+F 3 "https://www.dhgate.com/product/aml130a2402a-1-3-inch-240-240-round-tft-lcd/413771628.html#seo=WAP" H 6075 4625 60  0001 C CNN
+F 4 "AML130A2402A" H 6075 4625 60  0001 C CNN "MPN"
 	1    6075 4625
 	1    0    0    -1
